Commit message: Add RGB-D sensor to robot

File: src/map_my_world/urdf/my_robot.xacro (robot description, xacro)
@@ -1,5 +1,5 @@
 <?xml version="1.0"?>
 <robot name="my_robot" xmlns:xacro="http://www.ros.org/wiki/xacro">
-    <xacro:include filename="$(find where_am_i)/urdf/my_robot.gazebo" />
+    <xacro:include filename="$(find map_my_world)/urdf/my_robot.gazebo" />
     <link name="robot_footprint"/>
     <joint name="robot_footprint_joint" type="fixed">
@@ -201,5 +201,5 @@
             <origin xyz="0 0 0" rpy="0 0 0"/>
             <geometry>
-                <mesh filename="package://where_am_i/meshes/hokuyo.dae" />
+                <mesh filename="package://map_my_world/meshes/hokuyo.dae" />
             </geometry>
         </visual>
@@ -226,4 +226,12 @@
         <child link="hokuyo"/>
     </joint>
+    <!-- An RGB-D camera required for the RTAB-Map package -->
+    <link name="camera_link_optical">
+    </link>
+    <joint name="camera_optical_joint" type="fixed">
+        <origin xyz="0 0 0" rpy="-1.5707 0 -1.5707"/>
+        <parent link="camera"/>
+        <child link="camera_link_optical"/>
+    </joint>
     <gazebo reference="front_right_wheel">
         <material>Gazebo/DarkGrey</material>
